Commit message: Yayy! able to load controllers

File: robot_description/urdf/inc/ur5_macro.xacro (robot description, xacro)
@@ -42,5 +42,5 @@
      - Muhammad Asif Rana
   -->
-  <!-- <xacro:include filename="ur_transmissions.xacro"/> -->
+  <xacro:include filename="ur_transmissions.xacro"/>
   <xacro:include filename="ur_common.xacro"/>
   <xacro:macro name="ur_robot" params="
@@ -52,5 +52,6 @@
       safety_limits:=false
       safety_pos_margin:=0.15
-      safety_k_position:=20">
+      safety_k_position:=20
+      hw_interface">
   <!-- <xacro:arg name="mesh_path" default=""/> -->
     <!-- Load configuration data from the provided .yaml files -->
@@ -66,4 +67,5 @@
     <!-- Add URDF transmission elements (for ros_control) -->
     <!-- <xacro:ur_arm_transmission prefix="${prefix}"/> -->
+    <xacro:ur_arm_transmission prefix="${prefix}" hw_interface="${hw_interface}"/>
     <!-- links: main serial chain -->
     <link name="${prefix}base_link"/>

File: robot_description/urdf/inc/ur_transmissions.xacro (robot description, xacro)
@@ -1,14 +1,37 @@
 <?xml version="1.0"?>
 <robot xmlns:xacro="http://wiki.ros.org/xacro">
-  <!--
-    NOTE: the macro defined in this file is NOT part of the public API of this
-          package. Users CANNOT rely on this file being available, or stored in
-          this location. Nor can they rely on the existence of the macro.
-  -->
+  <!-- Macro for defining transmissions and ros2_control interface -->
+  <!-- <xacro:macro name="ur_arm_transmission" prefix="" hw_interface="PositionJointInterface"> -->
   <xacro:macro name="ur_arm_transmission" params="prefix hw_interface">
+    <!-- ros2_control interface for controlling the joint -->
+    <!-- ros2_control interface for controlling the joint -->
+    <ros2_control name="ur5_robot" type="system">
+      <hardware>
+          <plugin>fake_components/GenericSystem</plugin>
+      </hardware>
+      <joint name="shoulder_pan_joint">
+        <hardware_interface>PositionJointInterface</hardware_interface>
+      </joint>
+      <joint name="shoulder_lift_joint">
+        <hardware_interface>PositionJointInterface</hardware_interface>
+      </joint>
+      <joint name="elbow_joint">
+        <hardware_interface>PositionJointInterface</hardware_interface>
+      </joint>
+      <joint name="wrist_1_joint">
+        <hardware_interface>PositionJointInterface</hardware_interface>
+      </joint>
+      <joint name="wrist_2_joint">
+        <hardware_interface>PositionJointInterface</hardware_interface>
+      </joint>
+      <joint name="wrist_3_joint">
+        <hardware_interface>PositionJointInterface</hardware_interface>
+      </joint>
+    </ros2_control>
+    <!-- Transmission definition for each joint -->
     <transmission name="${prefix}shoulder_pan_trans">
       <type>transmission_interface/SimpleTransmission</type>
       <joint name="${prefix}shoulder_pan_joint">
-        <hardwareInterface>${hw_interface}</hardwareInterface>
+        <hardware_interface>${hw_interface}</hardware_interface>
       </joint>
       <actuator name="${prefix}shoulder_pan_motor">
@@ -19,5 +42,5 @@
       <type>transmission_interface/SimpleTransmission</type>
       <joint name="${prefix}shoulder_lift_joint">
-        <hardwareInterface>${hw_interface}</hardwareInterface>
+        <hardware_interface>${hw_interface}</hardware_interface>
       </joint>
       <actuator name="${prefix}shoulder_lift_motor">
@@ -28,5 +51,5 @@
       <type>transmission_interface/SimpleTransmission</type>
       <joint name="${prefix}elbow_joint">
-        <hardwareInterface>${hw_interface}</hardwareInterface>
+        <hardware_interface>${hw_interface}</hardware_interface>
       </joint>
       <actuator name="${prefix}elbow_motor">
@@ -34,8 +57,9 @@
       </actuator>
     </transmission>
+    <!-- Repeat for wrist joints -->
     <transmission name="${prefix}wrist_1_trans">
       <type>transmission_interface/SimpleTransmission</type>
       <joint name="${prefix}wrist_1_joint">
-        <hardwareInterface>${hw_interface}</hardwareInterface>
+        <hardware_interface>${hw_interface}</hardware_interface>
       </joint>
       <actuator name="${prefix}wrist_1_motor">
@@ -46,5 +70,5 @@
       <type>transmission_interface/SimpleTransmission</type>
       <joint name="${prefix}wrist_2_joint">
-        <hardwareInterface>${hw_interface}</hardwareInterface>
+        <hardware_interface>${hw_interface}</hardware_interface>
       </joint>
       <actuator name="${prefix}wrist_2_motor">
@@ -55,5 +79,5 @@
       <type>transmission_interface/SimpleTransmission</type>
       <joint name="${prefix}wrist_3_joint">
-        <hardwareInterface>${hw_interface}</hardwareInterface>
+        <hardware_interface>${hw_interface}</hardware_interface>
       </joint>
       <actuator name="${prefix}wrist_3_motor">

File: robot_description/urdf/ur5.urdf.xacro (robot description, xacro)
@@ -37,4 +37,5 @@
                   safety_limits="false"
                   safety_pos_margin="0.15"
-                  safety_k_position="20"/>
+                  safety_k_position="20"
+                  hw_interface="PositionJointInterface"/>
 </robot>

Commit message: Feature: Added ignition gazebo interface,          Added IgnitionSystem interface for controllers.
- Switched from fake_components/GenericSystem to ign_ros2_control/IgnitionSystem
  plugin. This is because fake_components/GenericSystem doesn't handle
  simulation of physical dynamics like gravity, inertia or friction.
- Able to load the controller

File: robot_description/urdf/inc/ur5_macro.xacro (robot description, xacro)
@@ -232,5 +232,5 @@
          <safety_controller soft_lower_limit="${shoulder_pan_lower_limit + safety_pos_margin}" soft_upper_limit="${shoulder_pan_upper_limit - safety_pos_margin}" k_position="${safety_k_position}" k_velocity="0.0"/>
       </xacro:if>
-      <dynamics damping="0" friction="0"/>
+      <dynamics damping="5.0" friction="2.0"/>
     </joint>
     <joint name="${prefix}shoulder_lift_joint" type="revolute">
@@ -244,5 +244,5 @@
          <safety_controller soft_lower_limit="${shoulder_lift_lower_limit + safety_pos_margin}" soft_upper_limit="${shoulder_lift_upper_limit - safety_pos_margin}" k_position="${safety_k_position}" k_velocity="0.0"/>
       </xacro:if>
-      <dynamics damping="0" friction="0"/>
+      <dynamics damping="5.0" friction="2.0"/>
     </joint>
     <joint name="${prefix}elbow_joint" type="revolute">
@@ -256,5 +256,5 @@
          <safety_controller soft_lower_limit="${elbow_joint_lower_limit + safety_pos_margin}" soft_upper_limit="${elbow_joint_upper_limit - safety_pos_margin}" k_position="${safety_k_position}" k_velocity="0.0"/>
       </xacro:if>
-      <dynamics damping="0" friction="0"/>
+      <dynamics damping="5.0" friction="2.0"/>
     </joint>
     <joint name="${prefix}wrist_1_joint" type="revolute">
@@ -268,5 +268,5 @@
          <safety_controller soft_lower_limit="${wrist_1_lower_limit + safety_pos_margin}" soft_upper_limit="${wrist_1_upper_limit - safety_pos_margin}" k_position="${safety_k_position}" k_velocity="0.0"/>
       </xacro:if>
-      <dynamics damping="0" friction="0"/>
+      <dynamics damping="5.0" friction="2.0"/>
     </joint>
     <joint name="${prefix}wrist_2_joint" type="revolute">
@@ -280,5 +280,5 @@
          <safety_controller soft_lower_limit="${wrist_2_lower_limit + safety_pos_margin}" soft_upper_limit="${wrist_2_upper_limit - safety_pos_margin}" k_position="${safety_k_position}" k_velocity="0.0"/>
       </xacro:if>
-      <dynamics damping="0" friction="0"/>
+      <dynamics damping="5.0" friction="2.0"/>
     </joint>
     <joint name="${prefix}wrist_3_joint" type="revolute">
@@ -292,5 +292,5 @@
          <safety_controller soft_lower_limit="${wrist_3_lower_limit + safety_pos_margin}" soft_upper_limit="${wrist_3_upper_limit - safety_pos_margin}" k_position="${safety_k_position}" k_velocity="0.0"/>
       </xacro:if>
-      <dynamics damping="0" friction="0"/>
+      <dynamics damping="5.0" friction="2.0"/>
     </joint>
     <!-- ROS-Industrial 'base' frame: base_link to UR 'Base' Coordinates transform -->

File: robot_description/urdf/inc/ur_transmissions.xacro (robot description, xacro)
@@ -1,42 +1,51 @@
 <?xml version="1.0"?>
 <robot xmlns:xacro="http://wiki.ros.org/xacro">
-  <!-- Macro for defining transmissions and ros2_control interface -->
-  <!-- <xacro:macro name="ur_arm_transmission" prefix="" hw_interface="PositionJointInterface"> -->
   <xacro:macro name="ur_arm_transmission" params="prefix hw_interface">
     <!-- ros2_control interface for controlling the joint -->
-    <!-- ros2_control interface for controlling the joint -->
-    <ros2_control name="ur5_robot" type="system">
+    <ros2_control name="IgnitionSystem" type="system">
       <hardware>
-          <plugin>fake_components/GenericSystem</plugin>
+          <plugin>ign_ros2_control/IgnitionSystem</plugin>
       </hardware>
       <joint name="shoulder_pan_joint">
         <hardware_interface>position</hardware_interface>
         <command_interface name="position"/>
-        <state_interface name="position"/>
+        <state_interface name="position">
+          <!-- <param name="initial_value">0.0</param> -->
+        </state_interface>
       </joint>
       <joint name="shoulder_lift_joint">
         <hardware_interface>position</hardware_interface>
         <command_interface name="position"/>
-        <state_interface name="position"/>
+        <state_interface name="position">
+          <!-- <param name="initial_value">0.0</param> -->
+        </state_interface>
       </joint>
       <joint name="elbow_joint">
         <hardware_interface>position</hardware_interface>
         <command_interface name="position"/>
-        <state_interface name="position"/>
+        <state_interface name="position">
+          <!-- <param name="initial_value">0.0</param> -->
+        </state_interface>
       </joint>
       <joint name="wrist_1_joint">
         <hardware_interface>position</hardware_interface>
         <command_interface name="position"/>
-        <state_interface name="position"/>
+        <state_interface name="position">
+          <!-- <param name="initial_value">0.0</param> -->
+        </state_interface>
       </joint>
       <joint name="wrist_2_joint">
         <hardware_interface>position</hardware_interface>
         <command_interface name="position"/>
-        <state_interface name="position"/>
+        <state_interface name="position">
+          <!-- <param name="initial_value">0.0</param> -->
+        </state_interface>
       </joint>
       <joint name="wrist_3_joint">
         <hardware_interface>position</hardware_interface>
         <command_interface name="position"/>
-        <state_interface name="position"/>
+        <state_interface name="position">
+          <!-- <param name="initial_value">0.0</param> -->
+        </state_interface>
       </joint>
     </ros2_control>
@@ -98,3 +107,9 @@
     </transmission>
   </xacro:macro>
+  <gazebo>
+    <plugin filename="libign_ros2_control-system.so" name="ign_ros2_control::IgnitionROS2ControlPlugin">
+      <parameters>$(find robot_motion_planning)/config/controllers.yaml</parameters>
+      <controller_manager_name>controller_manager</controller_manager_name>
+    </plugin>
+  </gazebo>
 </robot>
